File: kicad/ble.kicad_sch (KiCad schematic)
At the start: 12 parts, among them J6 Conn_Coaxial, U16 NRF52832-QFAA-R, Y1 32MHz

Commit message: checking shunt footprints
Parts:
- renumbered C64 to C61, C57 to C62, C59 to C63, C60 to C64, C58 to C65, C61 to C66, C62 to C67, C63 to C68, J6 to J10, Y1 to Y2
Connections:
- net BLE_RX: now also U16.4 (P0_02/AIN0); no longer U16.3 (P0_01/XL2)
- net BLE_TX: now also U16.3 (P0_01/XL2); no longer U16.2 (P0_00/XL1)
Other:
- moved on the sheet: C62, C65
Changed lines of the file:
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@@
 	)
 	(junction
-		(at 49.53 60.96)
+		(at 53.34 60.96)
 		(diameter 0)
 		(color 0 0 0 0)
@@
 	)
 	(no_connect
-		(at 109.22 87.63)
+		(at 109.22 82.55)
 	)
 	(no_connect
@@
 	(wire
 		(pts
-			(xy 49.53 60.96) (xy 49.53 64.77)
+			(xy 53.34 60.96) (xy 53.34 64.77)
 		)
 		(stroke
@@
 	(wire
 		(pts
-			(xy 53.34 60.96) (xy 49.53 60.96)
+			(xy 57.15 60.96) (xy 53.34 60.96)
 		)
 		(stroke
@@
 	(wire
 		(pts
-			(xy 60.96 60.96) (xy 77.47 60.96)
+			(xy 64.77 60.96) (xy 77.47 60.96)
 		)
 		(stroke
@@
 	(wire
 		(pts
-			(xy 60.96 45.72) (xy 77.47 45.72)
+			(xy 64.77 45.72) (xy 77.47 45.72)
 		)
 		(stroke
@@
 	(wire
 		(pts
-			(xy 53.34 45.72) (xy 49.53 45.72)
+			(xy 57.15 45.72) (xy 53.34 45.72)
 		)
 		(stroke
@@
 	(wire
 		(pts
-			(xy 49.53 45.72) (xy 49.53 60.96)
+			(xy 53.34 45.72) (xy 53.34 60.96)
 		)
 		(stroke
@@
 	(hierarchical_label "BLE_TX"
 		(shape output)
-		(at 109.22 82.55 180)
+		(at 109.22 85.09 180)
 		(effects
 			(font
@@
 	(hierarchical_label "BLE_RX"
 		(shape input)
-		(at 109.22 85.09 180)
+		(at 109.22 87.63 180)
 		(effects
 			(font
@@
 		(dnp no)
 		(fields_autoplaced yes)
-		(property "Reference" "J6"
+		(property "Reference" "J10"
 			(at 209.55 79.0331 0)
 			(effects
@@
 			(project ""
 				(path "/83aea3b7-5b9b-498e-8d41-e84fae2f87fa/7fcb459e-6347-48a4-bd99-c80bd89cbe59"
-					(reference "J6")
+					(reference "J10")
 					(unit 1)
 				)
@@
 		(dnp no)
 		(fields_autoplaced yes)
-		(property "Reference" "#PWR090"
+		(property "Reference" "#PWR098"
 			(at 205.74 99.06 0)
 			(effects
@@
 			(project "resc"
 				(path "/83aea3b7-5b9b-498e-8d41-e84fae2f87fa/7fcb459e-6347-48a4-bd99-c80bd89cbe59"
-					(reference "#PWR090")
+					(reference "#PWR098")
 					(unit 1)
 				)
@@
 		(on_board yes)
 		(dnp no)
-		(property "Reference" "C60"
+		(property "Reference" "C64"
 			(at 182.626 54.356 90)
 			(effects
@@
 			(project "resc"
 				(path "/83aea3b7-5b9b-498e-8d41-e84fae2f87fa/7fcb459e-6347-48a4-bd99-c80bd89cbe59"
-					(reference "C60")
+					(reference "C64")
 					(unit 1)
 				)
@@
 		(on_board yes)
 		(dnp no)
-		(property "Reference" "#PWR084"
+		(property "Reference" "#PWR094"
 			(at 85.09 60.96 0)
 			(effects
@@
 			(project "resc"
 				(path "/83aea3b7-5b9b-498e-8d41-e84fae2f87fa/7fcb459e-6347-48a4-bd99-c80bd89cbe59"
-					(reference "#PWR084")
+					(reference "#PWR094")
 					(unit 1)
 				)
@@
 		(on_board yes)
 		(dnp no)
-		(property "Reference" "C62"
+		(property "Reference" "C67"
 			(at 182.626 69.596 90)
 			(effects
@@
 			(project "resc"
 				(path "/83aea3b7-5b9b-498e-8d41-e84fae2f87fa/7fcb459e-6347-48a4-bd99-c80bd89cbe59"
-					(reference "C62")
+					(reference "C67")
 					(unit 1)
 				)
@@
 		(on_board yes)
 		(dnp no)
-		(property "Reference" "C61"
+		(property "Reference" "C66"
 			(at 182.626 61.976 90)
 			(effects
@@
 			(project "resc"
 				(path "/83aea3b7-5b9b-498e-8d41-e84fae2f87fa/7fcb459e-6347-48a4-bd99-c80bd89cbe59"
-					(reference "C61")
+					(reference "C66")
 					(unit 1)
 				)
@@
 		(dnp no)
 		(fields_autoplaced yes)
-		(property "Reference" "#PWR085"
+		(property "Reference" "#PWR099"
 			(at 172.72 144.78 0)
 			(effects
@@
 			(project ""
 				(path "/83aea3b7-5b9b-498e-8d41-e84fae2f87fa/7fcb459e-6347-48a4-bd99-c80bd89cbe59"
-					(reference "#PWR085")
+					(reference "#PWR099")
 					(unit 1)
 				)
@@
 		(on_board yes)
 		(dnp no)
-		(property "Reference" "#PWR099"
+		(property "Reference" "#PWR093"
 			(at 69.85 60.96 0)
 			(effects
@@
 			(project "resc"
 				(path "/83aea3b7-5b9b-498e-8d41-e84fae2f87fa/7fcb459e-6347-48a4-bd99-c80bd89cbe59"
-					(reference "#PWR099")
+					(reference "#PWR093")
 					(unit 1)
 				)
@@
 		(dnp no)
 		(fields_autoplaced yes)
-		(property "Reference" "#PWR086"
+		(property "Reference" "#PWR091"
 			(at 185.42 36.83 0)
 			(effects
@@
 			(project ""
 				(path "/83aea3b7-5b9b-498e-8d41-e84fae2f87fa/7fcb459e-6347-48a4-bd99-c80bd89cbe59"
-					(reference "#PWR086")
+					(reference "#PWR091")
 					(unit 1)
 				)
@@
 		(dnp no)
 		(fields_autoplaced yes)
-		(property "Reference" "C64"
+		(property "Reference" "C61"
 			(at 194.31 29.21 90)
 			(effects
@@
 			(project "resc"
 				(path "/83aea3b7-5b9b-498e-8d41-e84fae2f87fa/7fcb459e-6347-48a4-bd99-c80bd89cbe59"
-					(reference "C64")
+					(reference "C61")
 					(unit 1)
 				)
@@
 		(dnp no)
 		(fields_autoplaced yes)
-		(property "Reference" "#PWR087"
+		(property "Reference" "#PWR092"
 			(at 201.93 58.42 0)
 			(effects
@@
 			(project ""
 				(path "/83aea3b7-5b9b-498e-8d41-e84fae2f87fa/7fcb459e-6347-48a4-bd99-c80bd89cbe59"
-					(reference "#PWR087")
+					(reference "#PWR092")
 					(unit 1)
 				)
@@
 		(dnp no)
 		(fields_autoplaced yes)
-		(property "Reference" "C59"
+		(property "Reference" "C63"
 			(at 194.31 41.91 90)
 			(effects
@@
 			(project ""
 				(path "/83aea3b7-5b9b-498e-8d41-e84fae2f87fa/7fcb459e-6347-48a4-bd99-c80bd89cbe59"
-					(reference "C59")
+					(reference "C63")
 					(unit 1)
 				)
@@
 		(dnp no)
 		(fields_autoplaced yes)
-		(property "Reference" "C63"
+		(property "Reference" "C68"
 			(at 187.96 85.0899 0)
 			(effects
@@
 			(project ""
 				(path "/83aea3b7-5b9b-498e-8d41-e84fae2f87fa/7fcb459e-6347-48a4-bd99-c80bd89cbe59"
-					(reference "C63")
+					(reference "C68")
 					(unit 1)
 				)
@@
 	(symbol
 		(lib_id "power:GND")
-		(at 49.53 64.77 0)
+		(at 53.34 64.77 0)
 		(unit 1)
 		(exclude_from_sim no)
@@
 		(dnp no)
 		(fields_autoplaced yes)
-		(property "Reference" "#PWR083"
-			(at 49.53 71.12 0)
+		(property "Reference" "#PWR096"
+			(at 53.34 71.12 0)
 			(effects
 				(font
@@
 		)
 		(property "Value" "GND"
-			(at 49.53 69.85 0)
+			(at 53.34 69.85 0)
 			(effects
 				(font
@@
 		)
 		(property "Footprint" ""
-			(at 49.53 64.77 0)
+			(at 53.34 64.77 0)
 			(effects
 				(font
@@
 		)
 		(property "Datasheet" ""
-			(at 49.53 64.77 0)
+			(at 53.34 64.77 0)
 			(effects
 				(font
@@
 		)
 		(property "Description" "Power symbol creates a global label with name \"GND\" , ground"
-			(at 49.53 64.77 0)
+			(at 53.34 64.77 0)
 			(effects
 				(font
@@
 			(project ""
 				(path "/83aea3b7-5b9b-498e-8d41-e84fae2f87fa/7fcb459e-6347-48a4-bd99-c80bd89cbe59"
-					(reference "#PWR083")
+					(reference "#PWR096")
 					(unit 1)
 				)
@@
 		(dnp no)
 		(fields_autoplaced yes)
-		(property "Reference" "Y1"
+		(property "Reference" "Y2"
 			(at 86.36 48.3868 90)
 			(effects
@@
 			(project ""
 				(path "/83aea3b7-5b9b-498e-8d41-e84fae2f87fa/7fcb459e-6347-48a4-bd99-c80bd89cbe59"
-					(reference "Y1")
+					(reference "Y2")
 					(unit 1)
 				)
@@
 	(symbol
 		(lib_id "Device:C")
-		(at 57.15 45.72 90)
+		(at 60.96 45.72 90)
 		(unit 1)
 		(exclude_from_sim no)
@@
 		(dnp no)
 		(fields_autoplaced yes)
-		(property "Reference" "C57"
-			(at 57.15 38.1 90)
+		(property "Reference" "C62"
+			(at 60.96 38.1 90)
 			(effects
 				(font
@@
 		)
 		(property "Value" "8pF"
-			(at 57.15 40.64 90)
+			(at 60.96 40.64 90)
 			(effects
 				(font
@@
 		)
 		(property "Footprint" "Capacitor_SMD:C_0402_1005Metric"
-			(at 60.96 44.7548 0)
+			(at 64.77 44.7548 0)
 			(effects
 				(font
@@
 		)
 		(property "Datasheet" "~"
-			(at 57.15 45.72 0)
+			(at 60.96 45.72 0)
 			(effects
 				(font
@@
 		)
 		(property "Description" "Unpolarized capacitor"
-			(at 57.15 45.72 0)
+			(at 60.96 45.72 0)
 			(effects
 				(font
@@
 			(project ""
 				(path "/83aea3b7-5b9b-498e-8d41-e84fae2f87fa/7fcb459e-6347-48a4-bd99-c80bd89cbe59"
-					(reference "C57")
+					(reference "C62")
 					(unit 1)
 				)
@@
 		(dnp no)
 		(fields_autoplaced yes)
-		(property "Reference" "#PWR088"
+		(property "Reference" "#PWR097"
 			(at 184.15 99.06 0)
 			(effects
@@
 			(project "resc"
 				(path "/83aea3b7-5b9b-498e-8d41-e84fae2f87fa/7fcb459e-6347-48a4-bd99-c80bd89cbe59"
-					(reference "#PWR088")
+					(reference "#PWR097")
 					(unit 1)
 				)
@@
 		(dnp no)
 		(fields_autoplaced yes)
-		(property "Reference" "#PWR089"
+		(property "Reference" "#PWR095"
 			(at 196.85 63.5 0)
 			(effects
@@
 			(project "resc"
 				(path "/83aea3b7-5b9b-498e-8d41-e84fae2f87fa/7fcb459e-6347-48a4-bd99-c80bd89cbe59"
-					(reference "#PWR089")
+					(reference "#PWR095")
 					(unit 1)
 				)
@@
 	(symbol
 		(lib_id "Device:C")
-		(at 57.15 60.96 90)
+		(at 60.96 60.96 90)
 		(unit 1)
 		(exclude_from_sim no)
@@
 		(dnp no)
 		(fields_autoplaced yes)
-		(property "Reference" "C58"
-			(at 57.15 53.34 90)
+		(property "Reference" "C65"
+			(at 60.96 53.34 90)
 			(effects
 				(font
@@
 		)
 		(property "Value" "8pF"
-			(at 57.15 55.88 90)
+			(at 60.96 55.88 90)
 			(effects
 				(font
@@
 		)
 		(property "Footprint" "Capacitor_SMD:C_0402_1005Metric"
-			(at 60.96 59.9948 0)
+			(at 64.77 59.9948 0)
 			(effects
 				(font
@@
 		)
 		(property "Datasheet" "~"
-			(at 57.15 60.96 0)
+			(at 60.96 60.96 0)
 			(effects
 				(font
@@
 		)
 		(property "Description" "Unpolarized capacitor"
-			(at 57.15 60.96 0)
+			(at 60.96 60.96 0)
 			(effects
 				(font
@@
 			(project "resc"
 				(path "/83aea3b7-5b9b-498e-8d41-e84fae2f87fa/7fcb459e-6347-48a4-bd99-c80bd89cbe59"
-					(reference "C58")
+					(reference "C65")
 					(unit 1)
 				)

Commit message: routing gate driver
Parts:
- renumbered C61 to C58, C62 to C59, C63 to C60, C64 to C61, C65 to C62, C66 to C63, C67 to C64, C68 to C65
Changed lines of the file:
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@@
 		(title "rESC")
 		(date "2025-05-24")
-		(rev "a")
+		(rev "1")
 		(company "Tyler Lindsay")
 	)
@@
 		(on_board yes)
 		(dnp no)
-		(property "Reference" "C64"
+		(property "Reference" "C61"
 			(at 182.626 54.356 90)
 			(effects
@@
 			(project "resc"
 				(path "/83aea3b7-5b9b-498e-8d41-e84fae2f87fa/7fcb459e-6347-48a4-bd99-c80bd89cbe59"
-					(reference "C64")
+					(reference "C61")
 					(unit 1)
 				)
@@
 		(on_board yes)
 		(dnp no)
-		(property "Reference" "C67"
+		(property "Reference" "C64"
 			(at 182.626 69.596 90)
 			(effects
@@
 			(project "resc"
 				(path "/83aea3b7-5b9b-498e-8d41-e84fae2f87fa/7fcb459e-6347-48a4-bd99-c80bd89cbe59"
-					(reference "C67")
+					(reference "C64")
 					(unit 1)
 				)
@@
 		(on_board yes)
 		(dnp no)
-		(property "Reference" "C66"
+		(property "Reference" "C63"
 			(at 182.626 61.976 90)
 			(effects
@@
 			(project "resc"
 				(path "/83aea3b7-5b9b-498e-8d41-e84fae2f87fa/7fcb459e-6347-48a4-bd99-c80bd89cbe59"
-					(reference "C66")
+					(reference "C63")
 					(unit 1)
 				)
@@
 		(dnp no)
 		(fields_autoplaced yes)
-		(property "Reference" "C61"
+		(property "Reference" "C58"
 			(at 194.31 29.21 90)
 			(effects
@@
 			(project "resc"
 				(path "/83aea3b7-5b9b-498e-8d41-e84fae2f87fa/7fcb459e-6347-48a4-bd99-c80bd89cbe59"
-					(reference "C61")
+					(reference "C58")
 					(unit 1)
 				)
@@
 		(dnp no)
 		(fields_autoplaced yes)
-		(property "Reference" "C63"
+		(property "Reference" "C60"
 			(at 194.31 41.91 90)
 			(effects
@@
 			(project ""
 				(path "/83aea3b7-5b9b-498e-8d41-e84fae2f87fa/7fcb459e-6347-48a4-bd99-c80bd89cbe59"
-					(reference "C63")
+					(reference "C60")
 					(unit 1)
 				)
@@
 		(dnp no)
 		(fields_autoplaced yes)
-		(property "Reference" "C68"
+		(property "Reference" "C65"
 			(at 187.96 85.0899 0)
 			(effects
@@
 			(project ""
 				(path "/83aea3b7-5b9b-498e-8d41-e84fae2f87fa/7fcb459e-6347-48a4-bd99-c80bd89cbe59"
-					(reference "C68")
+					(reference "C65")
 					(unit 1)
 				)
@@
 		(dnp no)
 		(fields_autoplaced yes)
-		(property "Reference" "C62"
+		(property "Reference" "C59"
 			(at 60.96 38.1 90)
 			(effects
@@
 			(project ""
 				(path "/83aea3b7-5b9b-498e-8d41-e84fae2f87fa/7fcb459e-6347-48a4-bd99-c80bd89cbe59"
-					(reference "C62")
+					(reference "C59")
 					(unit 1)
 				)
@@
 		(dnp no)
 		(fields_autoplaced yes)
-		(property "Reference" "C65"
+		(property "Reference" "C62"
 			(at 60.96 53.34 90)
 			(effects
@@
 			(project "resc"
 				(path "/83aea3b7-5b9b-498e-8d41-e84fae2f87fa/7fcb459e-6347-48a4-bd99-c80bd89cbe59"
-					(reference "C65")
+					(reference "C62")
 					(unit 1)
 				)

Commit message: revert to v6.05
Other:
- moved on the sheet: C61, C63, C64
Changed lines of the file:
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@@
-	)
-	(junction
-		(at 187.96 63.5)
-		(diameter 0)
-		(color 0 0 0 0)
 	)
 	(junction
@@
 	)
 	(junction
+		(at 187.96 64.77)
+		(diameter 0)
+		(color 0 0 0 0)
+	)
+	(junction
 		(at 170.18 49.53)
 		(diameter 0)
@@
 	(wire
 		(pts
-			(xy 171.45 64.77) (xy 170.18 64.77)
+			(xy 170.18 64.77) (xy 175.26 64.77)
 		)
 		(stroke
@@
 	(wire
 		(pts
-			(xy 187.96 63.5) (xy 187.96 71.12)
+			(xy 187.96 57.15) (xy 187.96 64.77)
 		)
 		(stroke
@@
 	(wire
 		(pts
-			(xy 171.45 63.5) (xy 171.45 64.77)
-		)
-		(stroke
-			(width 0)
-			(type default)
-		)
-	)
-	(wire
-		(pts
 			(xy 69.85 53.34) (xy 69.85 54.61)
 		)
@@
 	(wire
 		(pts
-			(xy 171.45 71.12) (xy 175.26 71.12)
-		)
-		(stroke
-			(width 0)
-			(type default)
-		)
-	)
-	(wire
-		(pts
-			(xy 182.88 55.88) (xy 187.96 55.88)
-		)
-		(stroke
-			(width 0)
-			(type default)
-		)
-	)
-	(wire
-		(pts
-			(xy 171.45 67.31) (xy 171.45 71.12)
+			(xy 187.96 64.77) (xy 187.96 72.39)
+		)
+		(stroke
+			(width 0)
+			(type default)
+		)
+	)
+	(wire
+		(pts
+			(xy 172.72 72.39) (xy 175.26 72.39)
+		)
+		(stroke
+			(width 0)
+			(type default)
+		)
+	)
+	(wire
+		(pts
+			(xy 182.88 57.15) (xy 187.96 57.15)
+		)
+		(stroke
+			(width 0)
+			(type default)
+		)
+	)
+	(wire
+		(pts
+			(xy 172.72 67.31) (xy 172.72 72.39)
 		)
 		(stroke
@@
 	(wire
 		(pts
-			(xy 171.45 55.88) (xy 175.26 55.88)
+			(xy 172.72 57.15) (xy 175.26 57.15)
 		)
 		(stroke
@@
 	(wire
 		(pts
-			(xy 182.88 71.12) (xy 187.96 71.12)
+			(xy 182.88 72.39) (xy 187.96 72.39)
 		)
 		(stroke
@@
 	(wire
 		(pts
-			(xy 77.47 45.72) (xy 90.17 45.72)
-		)
-		(stroke
-			(width 0)
-			(type default)
-		)
-	)
-	(wire
-		(pts
-			(xy 171.45 59.69) (xy 170.18 59.69)
+			(xy 77.47 45.72) (xy 100.33 45.72)
+		)
+		(stroke
+			(width 0)
+			(type default)
+		)
+	)
+	(wire
+		(pts
+			(xy 172.72 59.69) (xy 170.18 59.69)
 		)
 		(stroke
@@
 	(wire
 		(pts
-			(xy 182.88 63.5) (xy 187.96 63.5)
+			(xy 182.88 64.77) (xy 187.96 64.77)
 		)
 		(stroke
@@
 	(wire
 		(pts
-			(xy 187.96 55.88) (xy 187.96 63.5)
-		)
-		(stroke
-			(width 0)
-			(type default)
-		)
-	)
-	(wire
-		(pts
-			(xy 171.45 63.5) (xy 175.26 63.5)
-		)
-		(stroke
-			(width 0)
-			(type default)
-		)
-	)
-	(wire
-		(pts
-			(xy 90.17 67.31) (xy 109.22 67.31)
-		)
-		(stroke
-			(width 0)
-			(type default)
-		)
-	)
-	(wire
-		(pts
-			(xy 170.18 67.31) (xy 171.45 67.31)
+			(xy 100.33 67.31) (xy 109.22 67.31)
+		)
+		(stroke
+			(width 0)
+			(type default)
+		)
+	)
+	(wire
+		(pts
+			(xy 170.18 67.31) (xy 172.72 67.31)
 		)
 		(stroke
@@
 	(wire
 		(pts
-			(xy 171.45 55.88) (xy 171.45 59.69)
+			(xy 172.72 57.15) (xy 172.72 59.69)
 		)
 		(stroke
@@
 	(wire
 		(pts
-			(xy 187.96 63.5) (xy 190.5 63.5)
+			(xy 187.96 64.77) (xy 190.5 64.77)
 		)
 		(stroke
@@
 	(wire
 		(pts
-			(xy 90.17 67.31) (xy 90.17 45.72)
+			(xy 100.33 67.31) (xy 100.33 45.72)
 		)
 		(stroke
@@
 	(symbol
 		(lib_id "Device:C")
-		(at 179.07 55.88 270)
+		(at 179.07 57.15 270)
 		(unit 1)
 		(exclude_from_sim no)
@@
 		(dnp no)
 		(property "Reference" "C61"
-			(at 182.626 54.356 90)
+			(at 182.626 55.626 90)
 			(effects
 				(font
@@
 		)
 		(property "Value" "4.7uF"
-			(at 183.388 57.15 90)
+			(at 183.388 58.42 90)
 			(effects
 				(font
@@
 		)
 		(property "Footprint" "Capacitor_SMD:C_0402_1005Metric"
-			(at 175.26 56.8452 0)
+			(at 175.26 58.1152 0)
 			(effects
 				(font
@@
 		)
 		(property "Datasheet" "~"
-			(at 179.07 55.88 0)
+			(at 179.07 57.15 0)
 			(effects
 				(font
@@
 		)
 		(property "Description" "Unpolarized capacitor"
-			(at 179.07 55.88 0)
+			(at 179.07 57.15 0)
 			(effects
 				(font
@@
 	(symbol
 		(lib_id "Device:C")
-		(at 179.07 71.12 270)
+		(at 179.07 72.39 270)
 		(unit 1)
 		(exclude_from_sim no)
@@
 		(dnp no)
 		(property "Reference" "C64"
-			(at 182.626 69.596 90)
+			(at 182.626 70.866 90)
 			(effects
 				(font
@@
 		)
 		(property "Value" "1uF"
-			(at 182.626 72.39 90)
+			(at 182.626 73.66 90)
 			(effects
 				(font
@@
 		)
 		(property "Footprint" "Capacitor_SMD:C_0402_1005Metric"
-			(at 175.26 72.0852 0)
+			(at 175.26 73.3552 0)
 			(effects
 				(font
@@
 		)
 		(property "Datasheet" "~"
-			(at 179.07 71.12 0)
+			(at 179.07 72.39 0)
 			(effects
 				(font
@@
 		)
 		(property "Description" "Unpolarized capacitor"
-			(at 179.07 71.12 0)
+			(at 179.07 72.39 0)
 			(effects
 				(font
@@
 	(symbol
 		(lib_id "Device:C")
-		(at 179.07 63.5 270)
+		(at 179.07 64.77 270)
 		(unit 1)
 		(exclude_from_sim no)
@@
 		(dnp no)
 		(property "Reference" "C63"
-			(at 182.626 61.976 90)
+			(at 182.626 63.246 90)
 			(effects
 				(font
@@
 		)
 		(property "Value" "100pF"
-			(at 183.388 64.77 90)
+			(at 183.388 66.04 90)
 			(effects
 				(font
@@
 		)
 		(property "Footprint" "Capacitor_SMD:C_0402_1005Metric"
-			(at 175.26 64.4652 0)
+			(at 175.26 65.7352 0)
 			(effects
 				(font
@@
 		)
 		(property "Datasheet" "~"
-			(at 179.07 63.5 0)
+			(at 179.07 64.77 0)
 			(effects
 				(font
@@
 		)
 		(property "Description" "Unpolarized capacitor"
-			(at 179.07 63.5 0)
+			(at 179.07 64.77 0)
 			(effects
 				(font
@@
 	(symbol
 		(lib_id "power:GND")
-		(at 190.5 63.5 90)
+		(at 190.5 64.77 90)
 		(unit 1)
 		(exclude_from_sim no)
@@
 		(fields_autoplaced yes)
 		(property "Reference" "#PWR095"
-			(at 196.85 63.5 0)
+			(at 196.85 64.77 0)
 			(effects
 				(font
@@
 		)
 		(property "Value" "GND"
-			(at 194.31 63.4999 90)
+			(at 194.31 64.7699 90)
 			(effects
 				(font
@@
 		)
 		(property "Footprint" ""
-			(at 190.5 63.5 0)
+			(at 190.5 64.77 0)
 			(effects
 				(font
@@
 		)
 		(property "Datasheet" ""
-			(at 190.5 63.5 0)
+			(at 190.5 64.77 0)
 			(effects
 				(font
@@
 		)
 		(property "Description" "Power symbol creates a global label with name \"GND\" , ground"
-			(at 190.5 63.5 0)
-			(effects
-				(font
+			(at 190.5 64.77 0)
+			(effects
+				(font
