File: kicad/can.kicad_sch (KiCad schematic)
At the start: 4 parts, among them U3 TJA1051T-3

Commit message: checking shunt footprints
Parts:
- renumbered C1 to C16, C2 to C17, R1 to R18, U3 to U2
Changed lines of the file:
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@@
 		(dnp no)
 		(fields_autoplaced yes)
-		(property "Reference" "#PWR02"
+		(property "Reference" "#PWR038"
 			(at 139.7 125.73 0)
 			(effects
@@
 			(project "resc"
 				(path "/83aea3b7-5b9b-498e-8d41-e84fae2f87fa/1a126724-f6f9-4d54-8180-2481aea43f13"
-					(reference "#PWR02")
+					(reference "#PWR038")
 					(unit 1)
 				)
@@
 		(dnp no)
 		(fields_autoplaced yes)
-		(property "Reference" "#PWR01"
+		(property "Reference" "#PWR036"
 			(at 139.7 81.28 0)
 			(effects
@@
 			(project "resc"
 				(path "/83aea3b7-5b9b-498e-8d41-e84fae2f87fa/1a126724-f6f9-4d54-8180-2481aea43f13"
-					(reference "#PWR01")
+					(reference "#PWR036")
 					(unit 1)
 				)
@@
 		(dnp no)
 		(fields_autoplaced yes)
-		(property "Reference" "U3"
+		(property "Reference" "U2"
 			(at 141.8433 88.9 0)
 			(effects
@@
 			(project "resc"
 				(path "/83aea3b7-5b9b-498e-8d41-e84fae2f87fa/1a126724-f6f9-4d54-8180-2481aea43f13"
-					(reference "U3")
+					(reference "U2")
 					(unit 1)
 				)
@@
 		(dnp no)
 		(fields_autoplaced yes)
-		(property "Reference" "C2"
+		(property "Reference" "C17"
 			(at 120.65 109.2199 0)
 			(effects
@@
 			(project "resc"
 				(path "/83aea3b7-5b9b-498e-8d41-e84fae2f87fa/1a126724-f6f9-4d54-8180-2481aea43f13"
-					(reference "C2")
+					(reference "C17")
 					(unit 1)
 				)
@@
 		(dnp no)
 		(fields_autoplaced yes)
-		(property "Reference" "#PWR03"
+		(property "Reference" "#PWR037"
 			(at 116.84 106.68 0)
 			(effects
@@
 			(project "resc"
 				(path "/83aea3b7-5b9b-498e-8d41-e84fae2f87fa/1a126724-f6f9-4d54-8180-2481aea43f13"
-					(reference "#PWR03")
+					(reference "#PWR037")
 					(unit 1)
 				)
@@
 		(dnp no)
 		(fields_autoplaced yes)
-		(property "Reference" "R1"
+		(property "Reference" "R18"
 			(at 171.45 100.3299 0)
 			(effects
@@
 			(project "resc"
 				(path "/83aea3b7-5b9b-498e-8d41-e84fae2f87fa/1a126724-f6f9-4d54-8180-2481aea43f13"
-					(reference "R1")
+					(reference "R18")
 					(unit 1)
 				)
@@
 		(dnp no)
 		(fields_autoplaced yes)
-		(property "Reference" "C1"
+		(property "Reference" "C16"
 			(at 166.37 83.8199 0)
 			(effects
@@
 			(project "resc"
 				(path "/83aea3b7-5b9b-498e-8d41-e84fae2f87fa/1a126724-f6f9-4d54-8180-2481aea43f13"
-					(reference "C1")
-					(unit 1)
-				)
+					(reference "C16")
+					(unit 1)
+				)

Commit message: gate driver routed to mosfets, working on misc stm32 related components
Connections:
- net VCC is gone; now on net +5V: C17.1, U2.5 (VIO)
Changed lines of the file:
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@@
+	)
+	(symbol
+		(lib_id "power:+5V")
+		(at 116.84 102.87 0)
+		(unit 1)
+		(exclude_from_sim no)
+		(in_bom yes)
+		(on_board yes)
+		(dnp no)
+		(fields_autoplaced yes)
+		(property "Reference" "#PWR037"
+			(at 116.84 106.68 0)
+			(effects
+				(font
+					(size 1.27 1.27)
+				)
+				(hide yes)
+			)
+		)
+		(property "Value" "+5V"
+			(at 116.84 97.79 0)
+			(effects
+				(font
+					(size 1.27 1.27)
+				)
+			)
+		)
+		(property "Footprint" ""
+			(at 116.84 102.87 0)
+			(effects
+				(font
+					(size 1.27 1.27)
+				)
+				(hide yes)
+			)
+		)
+		(property "Datasheet" ""
+			(at 116.84 102.87 0)
+			(effects
+				(font
+					(size 1.27 1.27)
+				)
+				(hide yes)
+			)
+		)
+		(property "Description" "Power symbol creates a global label with name \"+5V\""
+			(at 116.84 102.87 0)
+			(effects
+				(font
+					(size 1.27 1.27)
+				)
+				(hide yes)
+			)
+		)
+		(pin "1"
+		)
+		(instances
+			(project ""
+				(path "/83aea3b7-5b9b-498e-8d41-e84fae2f87fa/1a126724-f6f9-4d54-8180-2481aea43f13"
+					(reference "#PWR037")
+					(unit 1)
+				)
+			)
+		)
 	)
 	(symbol
@@
 					(unit 1)
 				)
-			)
-		)
-	)
-	(symbol
-		(lib_id "power:VCC")
-		(at 116.84 102.87 0)
-		(unit 1)
-		(exclude_from_sim no)
-		(in_bom yes)
-		(on_board yes)
-		(dnp no)
-		(fields_autoplaced yes)
-		(property "Reference" "#PWR037"
-			(at 116.84 106.68 0)
-			(effects
-				(font
-					(size 1.27 1.27)
-				)
-				(hide yes)
-			)
-		)
-		(property "Value" "VCC"
-			(at 116.84 97.79 0)
-			(effects
-				(font
-					(size 1.27 1.27)
-				)
-			)
-		)
-		(property "Footprint" ""
-			(at 116.84 102.87 0)
-			(effects
-				(font
-					(size 1.27 1.27)
-				)
-				(hide yes)
-			)
-		)
-		(property "Datasheet" ""
-			(at 116.84 102.87 0)
-			(effects
-				(font
-					(size 1.27 1.27)
-				)
-				(hide yes)
-			)
-		)
-		(property "Description" "Power symbol creates a global label with name \"VCC\""
-			(at 116.84 102.87 0)
-			(effects
-				(font
-					(size 1.27 1.27)
-				)
-				(hide yes)
-			)
-		)
-		(pin "1"
-		)
-		(instances
-			(project "resc"
-				(path "/83aea3b7-5b9b-498e-8d41-e84fae2f87fa/1a126724-f6f9-4d54-8180-2481aea43f13"
-					(reference "#PWR037")
-					(unit 1)
-				)

Commit message: gate driver mostly schematic'd and pcb started
Parts:
- renumbered C16 to C14, C17 to C15, R18 to R13
Changed lines of the file:
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@@
 		(dnp no)
 		(fields_autoplaced yes)
-		(property "Reference" "#PWR038"
+		(property "Reference" "#PWR033"
 			(at 139.7 125.73 0)
 			(effects
@@
 			(project "resc"
 				(path "/83aea3b7-5b9b-498e-8d41-e84fae2f87fa/1a126724-f6f9-4d54-8180-2481aea43f13"
-					(reference "#PWR038")
+					(reference "#PWR033")
 					(unit 1)
 				)
@@
 		(dnp no)
 		(fields_autoplaced yes)
-		(property "Reference" "#PWR036"
+		(property "Reference" "#PWR031"
 			(at 139.7 81.28 0)
 			(effects
@@
 			(project "resc"
 				(path "/83aea3b7-5b9b-498e-8d41-e84fae2f87fa/1a126724-f6f9-4d54-8180-2481aea43f13"
-					(reference "#PWR036")
+					(reference "#PWR031")
 					(unit 1)
 				)
@@
 		(dnp no)
 		(fields_autoplaced yes)
-		(property "Reference" "#PWR037"
+		(property "Reference" "#PWR032"
 			(at 116.84 106.68 0)
 			(effects
@@
 			(project ""
 				(path "/83aea3b7-5b9b-498e-8d41-e84fae2f87fa/1a126724-f6f9-4d54-8180-2481aea43f13"
-					(reference "#PWR037")
+					(reference "#PWR032")
 					(unit 1)
 				)
@@
 		(dnp no)
 		(fields_autoplaced yes)
-		(property "Reference" "C17"
+		(property "Reference" "C15"
 			(at 120.65 109.2199 0)
 			(effects
@@
 			(project "resc"
 				(path "/83aea3b7-5b9b-498e-8d41-e84fae2f87fa/1a126724-f6f9-4d54-8180-2481aea43f13"
-					(reference "C17")
+					(reference "C15")
 					(unit 1)
 				)
@@
 		(dnp no)
 		(fields_autoplaced yes)
-		(property "Reference" "R18"
+		(property "Reference" "R13"
 			(at 171.45 100.3299 0)
 			(effects
@@
 			(project "resc"
 				(path "/83aea3b7-5b9b-498e-8d41-e84fae2f87fa/1a126724-f6f9-4d54-8180-2481aea43f13"
-					(reference "R18")
+					(reference "R13")
 					(unit 1)
 				)
@@
 		(dnp no)
 		(fields_autoplaced yes)
-		(property "Reference" "C16"
+		(property "Reference" "C14"
 			(at 166.37 83.8199 0)
 			(effects
@@
 			(project "resc"
 				(path "/83aea3b7-5b9b-498e-8d41-e84fae2f87fa/1a126724-f6f9-4d54-8180-2481aea43f13"
-					(reference "C16")
-					(unit 1)
-				)
+					(reference "C14")
+					(unit 1)
+				)

Commit message: rev3 ordered
Parts:
- R18: renamed from R13; symbol Device:R -> Device:R_US
- renumbered C14 to C16, C15 to C17
Changed lines of the file:
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@@
 		(dnp no)
 		(fields_autoplaced yes)
-		(property "Reference" "#PWR033"
+		(property "Reference" "#PWR038"
 			(at 139.7 125.73 0)
 			(effects
@@
 			(project "resc"
 				(path "/83aea3b7-5b9b-498e-8d41-e84fae2f87fa/1a126724-f6f9-4d54-8180-2481aea43f13"
-					(reference "#PWR033")
+					(reference "#PWR038")
 					(unit 1)
 				)
@@
 		(dnp no)
 		(fields_autoplaced yes)
-		(property "Reference" "#PWR031"
+		(property "Reference" "#PWR036"
 			(at 139.7 81.28 0)
 			(effects
@@
 			(project "resc"
 				(path "/83aea3b7-5b9b-498e-8d41-e84fae2f87fa/1a126724-f6f9-4d54-8180-2481aea43f13"
-					(reference "#PWR031")
+					(reference "#PWR036")
 					(unit 1)
 				)
@@
 		(dnp no)
 		(fields_autoplaced yes)
-		(property "Reference" "#PWR032"
+		(property "Reference" "#PWR037"
 			(at 116.84 106.68 0)
 			(effects
@@
 			(project ""
 				(path "/83aea3b7-5b9b-498e-8d41-e84fae2f87fa/1a126724-f6f9-4d54-8180-2481aea43f13"
-					(reference "#PWR032")
+					(reference "#PWR037")
 					(unit 1)
 				)
@@
 		(dnp no)
 		(fields_autoplaced yes)
-		(property "Reference" "C15"
+		(property "Reference" "C17"
 			(at 120.65 109.2199 0)
 			(effects
@@
 			(project "resc"
 				(path "/83aea3b7-5b9b-498e-8d41-e84fae2f87fa/1a126724-f6f9-4d54-8180-2481aea43f13"
-					(reference "C15")
-					(unit 1)
-				)
-			)
-		)
-	)
-	(symbol
-		(lib_id "Device:R")
+					(reference "C17")
+					(unit 1)
+				)
+			)
+		)
+	)
+	(symbol
+		(lib_id "Device:R_US")
 		(at 168.91 101.6 0)
 		(unit 1)
@@
 		(dnp no)
 		(fields_autoplaced yes)
-		(property "Reference" "R13"
+		(property "Reference" "R18"
 			(at 171.45 100.3299 0)
 			(effects
@@
 		)
 		(property "Footprint" "Resistor_SMD:R_0402_1005Metric"
-			(at 167.132 101.6 90)
+			(at 169.926 101.854 90)
 			(effects
 				(font
@@
 			)
 		)
-		(property "Description" "Resistor"
+		(property "Description" "Resistor, US symbol"
 			(at 168.91 101.6 0)
 			(effects
@@
 			(project "resc"
 				(path "/83aea3b7-5b9b-498e-8d41-e84fae2f87fa/1a126724-f6f9-4d54-8180-2481aea43f13"
-					(reference "R13")
+					(reference "R18")
 					(unit 1)
 				)
@@
 		(dnp no)
 		(fields_autoplaced yes)
-		(property "Reference" "C14"
+		(property "Reference" "C16"
 			(at 166.37 83.8199 0)
 			(effects
@@
 			(project "resc"
 				(path "/83aea3b7-5b9b-498e-8d41-e84fae2f87fa/1a126724-f6f9-4d54-8180-2481aea43f13"
-					(reference "C14")
-					(unit 1)
-				)
+					(reference "C16")
+					(unit 1)
+				)
