File: kicad/mcu.kicad_sch (KiCad schematic)
At the start: 13 parts, among them U2 STM32F405RGTx, Y2 8MHz

Commit message: checking shunt footprints
Parts:
- renumbered C22 to C10, C15 to C11, C14 to C13, C13 to C14, C16 to C15, C17 to C5, C18 to C6, C19 to C7, C20 to C8, C21 to C9, U2 to U1, Y2 to Y1
Changed lines of the file:
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@@
 		(dnp no)
 		(fields_autoplaced yes)
-		(property "Reference" "C18"
+		(property "Reference" "C6"
 			(at 198.12 35.5599 0)
 			(effects
@@
 			(project "resc"
 				(path "/83aea3b7-5b9b-498e-8d41-e84fae2f87fa/b16235e1-cba7-448a-b9f5-6f75b6848b7e"
-					(reference "C18")
+					(reference "C6")
 					(unit 1)
 				)
@@
 		(dnp no)
 		(fields_autoplaced yes)
-		(property "Reference" "#PWR012"
+		(property "Reference" "#PWR032"
 			(at 125.73 69.85 0)
 			(effects
@@
 			(project "resc"
 				(path "/83aea3b7-5b9b-498e-8d41-e84fae2f87fa/b16235e1-cba7-448a-b9f5-6f75b6848b7e"
-					(reference "#PWR012")
+					(reference "#PWR032")
 					(unit 1)
 				)
@@
 		(dnp no)
 		(fields_autoplaced yes)
-		(property "Reference" "#PWR014"
+		(property "Reference" "#PWR035"
 			(at 151.13 156.21 0)
 			(effects
@@
 			(project "resc"
 				(path "/83aea3b7-5b9b-498e-8d41-e84fae2f87fa/b16235e1-cba7-448a-b9f5-6f75b6848b7e"
-					(reference "#PWR014")
+					(reference "#PWR035")
 					(unit 1)
 				)
@@
 		(dnp no)
 		(fields_autoplaced yes)
-		(property "Reference" "#PWR010"
+		(property "Reference" "#PWR031"
 			(at 114.3 63.5 0)
 			(effects
@@
 			(project "resc"
 				(path "/83aea3b7-5b9b-498e-8d41-e84fae2f87fa/b16235e1-cba7-448a-b9f5-6f75b6848b7e"
-					(reference "#PWR010")
+					(reference "#PWR031")
 					(unit 1)
 				)
@@
 		(dnp no)
 		(fields_autoplaced yes)
-		(property "Reference" "#PWR016"
+		(property "Reference" "#PWR029"
 			(at 187.96 46.99 0)
 			(effects
@@
 			(project "resc"
 				(path "/83aea3b7-5b9b-498e-8d41-e84fae2f87fa/b16235e1-cba7-448a-b9f5-6f75b6848b7e"
-					(reference "#PWR016")
+					(reference "#PWR029")
 					(unit 1)
 				)
@@
 		(dnp no)
 		(fields_autoplaced yes)
-		(property "Reference" "C20"
+		(property "Reference" "C8"
 			(at 223.52 35.5599 0)
 			(effects
@@
 			(project "resc"
 				(path "/83aea3b7-5b9b-498e-8d41-e84fae2f87fa/b16235e1-cba7-448a-b9f5-6f75b6848b7e"
-					(reference "C20")
+					(reference "C8")
 					(unit 1)
 				)
@@
 		(dnp no)
 		(fields_autoplaced yes)
-		(property "Reference" "C17"
+		(property "Reference" "C5"
 			(at 185.42 35.5599 0)
 			(effects
@@
 			(project "resc"
 				(path "/83aea3b7-5b9b-498e-8d41-e84fae2f87fa/b16235e1-cba7-448a-b9f5-6f75b6848b7e"
-					(reference "C17")
+					(reference "C5")
 					(unit 1)
 				)
@@
 		(dnp no)
 		(fields_autoplaced yes)
-		(property "Reference" "Y2"
+		(property "Reference" "Y1"
 			(at 86.36 64.77 0)
 			(effects
@@
 			(project "resc"
 				(path "/83aea3b7-5b9b-498e-8d41-e84fae2f87fa/b16235e1-cba7-448a-b9f5-6f75b6848b7e"
-					(reference "Y2")
+					(reference "Y1")
 					(unit 1)
 				)
@@
 		(dnp no)
 		(fields_autoplaced yes)
-		(property "Reference" "#PWR013"
+		(property "Reference" "#PWR030"
 			(at 151.13 54.61 0)
 			(effects
@@
 			(project "resc"
 				(path "/83aea3b7-5b9b-498e-8d41-e84fae2f87fa/b16235e1-cba7-448a-b9f5-6f75b6848b7e"
-					(reference "#PWR013")
+					(reference "#PWR030")
 					(unit 1)
 				)
@@
 		(dnp no)
 		(fields_autoplaced yes)
-		(property "Reference" "#PWR011"
+		(property "Reference" "#PWR034"
 			(at 114.3 144.78 0)
 			(effects
@@
 			(project "resc"
 				(path "/83aea3b7-5b9b-498e-8d41-e84fae2f87fa/b16235e1-cba7-448a-b9f5-6f75b6848b7e"
-					(reference "#PWR011")
+					(reference "#PWR034")
 					(unit 1)
 				)
@@
 		(dnp no)
 		(fields_autoplaced yes)
-		(property "Reference" "C14"
+		(property "Reference" "C13"
 			(at 99.06 74.9299 0)
 			(effects
@@
 			(project "resc"
 				(path "/83aea3b7-5b9b-498e-8d41-e84fae2f87fa/b16235e1-cba7-448a-b9f5-6f75b6848b7e"
-					(reference "C14")
+					(reference "C13")
 					(unit 1)
 				)
@@
 		(dnp no)
 		(fields_autoplaced yes)
-		(property "Reference" "C19"
+		(property "Reference" "C7"
 			(at 210.82 35.5599 0)
 			(effects
@@
 			(project "resc"
 				(path "/83aea3b7-5b9b-498e-8d41-e84fae2f87fa/b16235e1-cba7-448a-b9f5-6f75b6848b7e"
-					(reference "C19")
+					(reference "C7")
 					(unit 1)
 				)
@@
 		(dnp no)
 		(fields_autoplaced yes)
-		(property "Reference" "U2"
+		(property "Reference" "U1"
 			(at 154.5433 148.59 0)
 			(effects
@@
 			(project "resc"
 				(path "/83aea3b7-5b9b-498e-8d41-e84fae2f87fa/b16235e1-cba7-448a-b9f5-6f75b6848b7e"
-					(reference "U2")
+					(reference "U1")
 					(unit 1)
 				)
@@
 		(dnp no)
 		(fields_autoplaced yes)
-		(property "Reference" "C13"
+		(property "Reference" "C14"
 			(at 111.76 133.3499 0)
 			(effects
@@
 			(project "resc"
 				(path "/83aea3b7-5b9b-498e-8d41-e84fae2f87fa/b16235e1-cba7-448a-b9f5-6f75b6848b7e"
-					(reference "C13")
+					(reference "C14")
 					(unit 1)
 				)
@@
 		(dnp no)
 		(fields_autoplaced yes)
-		(property "Reference" "C21"
+		(property "Reference" "C9"
 			(at 236.22 35.5599 0)
 			(effects
@@
 			(project "resc"
 				(path "/83aea3b7-5b9b-498e-8d41-e84fae2f87fa/b16235e1-cba7-448a-b9f5-6f75b6848b7e"
-					(reference "C21")
+					(reference "C9")
 					(unit 1)
 				)
@@
 		(dnp no)
 		(fields_autoplaced yes)
-		(property "Reference" "C16"
+		(property "Reference" "C15"
 			(at 124.46 133.3499 0)
 			(effects
@@
 			(project "resc"
 				(path "/83aea3b7-5b9b-498e-8d41-e84fae2f87fa/b16235e1-cba7-448a-b9f5-6f75b6848b7e"
-					(reference "C16")
+					(reference "C15")
 					(unit 1)
 				)
@@
 		(dnp no)
 		(fields_autoplaced yes)
-		(property "Reference" "#PWR09"
+		(property "Reference" "#PWR033"
 			(at 86.36 90.17 0)
 			(effects
@@
 			(project "resc"
 				(path "/83aea3b7-5b9b-498e-8d41-e84fae2f87fa/b16235e1-cba7-448a-b9f5-6f75b6848b7e"
-					(reference "#PWR09")
+					(reference "#PWR033")
 					(unit 1)
 				)
@@
 		(dnp no)
 		(fields_autoplaced yes)
-		(property "Reference" "C22"
+		(property "Reference" "C10"
 			(at 248.92 35.5599 0)
 			(effects
@@
 			(project "resc"
 				(path "/83aea3b7-5b9b-498e-8d41-e84fae2f87fa/b16235e1-cba7-448a-b9f5-6f75b6848b7e"
-					(reference "C22")
+					(reference "C10")
 					(unit 1)
 				)
@@
 		(dnp no)
 		(fields_autoplaced yes)
-		(property "Reference" "C15"
+		(property "Reference" "C11"
 			(at 118.11 52.0699 0)
 			(effects
@@
 			(project "resc"
 				(path "/83aea3b7-5b9b-498e-8d41-e84fae2f87fa/b16235e1-cba7-448a-b9f5-6f75b6848b7e"
-					(reference "C15")
+					(reference "C11")
 					(unit 1)
 				)
@@
 		(dnp no)
 		(fields_autoplaced yes)
-		(property "Reference" "#PWR015"
+		(property "Reference" "#PWR028"
 			(at 187.96 36.83 0)
 			(effects
@@
 			(project "resc"
 				(path "/83aea3b7-5b9b-498e-8d41-e84fae2f87fa/b16235e1-cba7-448a-b9f5-6f75b6848b7e"
-					(reference "#PWR015")
-					(unit 1)
-				)
+					(reference "#PWR028")
+					(unit 1)
+				)

Commit message: working on fet fp
Parts:
- Y1: footprint Crystal:Crystal_SMD_2016-4Pin_2.0x1.6mm -> Crystal:Crystal_SMD_3225-4Pin_3.2x2.5mm
Changed lines of the file:
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@@
 			)
 		)
-		(property "Footprint" "Crystal:Crystal_SMD_2016-4Pin_2.0x1.6mm"
+		(property "Footprint" "Crystal:Crystal_SMD_3225-4Pin_3.2x2.5mm"
 			(at 86.36 72.39 0)
 			(effects

Commit message: gate driver routed to mosfets, working on misc stm32 related components
Parts:
- Y1: symbol Device:Crystal_GND3 -> Device:Crystal_GND24
Connections:
- net GND: now also Y1.2, Y1.4; no longer Y1.3
- net at C13.1, U1.6 (PH1): now also Y1.3; no longer Y1.2
Changed lines of the file:
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@@
+	)
+	(junction
+		(at 91.44 81.28)
+		(diameter 0)
+		(color 0 0 0 0)
 	)
 	(junction
@@
 	(wire
 		(pts
+			(xy 86.36 67.31) (xy 86.36 66.04)
+		)
+		(stroke
+			(width 0)
+			(type default)
+		)
+	)
+	(wire
+		(pts
 			(xy 120.65 128.27) (xy 120.65 130.81)
 		)
@@
 	(wire
 		(pts
+			(xy 91.44 81.28) (xy 86.36 81.28)
+		)
+		(stroke
+			(width 0)
+			(type default)
+		)
+	)
+	(wire
+		(pts
 			(xy 128.27 62.23) (xy 125.73 62.23)
 		)
@@
 	(wire
 		(pts
-			(xy 95.25 81.28) (xy 86.36 81.28)
+			(xy 95.25 81.28) (xy 91.44 81.28)
 		)
 		(stroke
@@
 	(wire
 		(pts
+			(xy 86.36 66.04) (xy 91.44 66.04)
+		)
+		(stroke
+			(width 0)
+			(type default)
+		)
+	)
+	(wire
+		(pts
 			(xy 107.95 138.43) (xy 114.3 138.43)
 		)
@@
 		(pts
 			(xy 219.71 40.64) (xy 232.41 40.64)
+		)
+		(stroke
+			(width 0)
+			(type default)
+		)
+	)
+	(wire
+		(pts
+			(xy 91.44 66.04) (xy 91.44 81.28)
 		)
 		(stroke
@@
 	)
 	(symbol
-		(lib_id "Device:Crystal_GND3")
+		(lib_id "Device:Crystal_GND24")
 		(at 86.36 72.39 0)
 		(unit 1)
@@
 		(on_board yes)
 		(dnp no)
-		(fields_autoplaced yes)
 		(property "Reference" "Y1"
-			(at 86.36 64.77 0)
+			(at 81.788 64.516 0)
 			(effects
 				(font
@@
 		)
 		(property "Value" "8MHz"
-			(at 86.36 67.31 0)
+			(at 81.788 67.056 0)
 			(effects
 				(font
@@
 			)
 		)
-		(property "Description" "Three pin crystal, GND on pin 3"
+		(property "Description" "Four pin crystal, GND on pins 2 and 4"
 			(at 86.36 72.39 0)
 			(effects
@@
 		(pin "2"
 		)
+		(pin "4"
+		)
 		(instances

Commit message: gate driver mostly schematic'd and pcb started
Parts:
- renumbered C12 to C10, C13 to C11, C14 to C12, C15 to C13, C5 to C3, C6 to C4, C7 to C5, C8 to C6, C9 to C7, C10 to C8, C11 to C9
Connections:
- net LED2: no longer names the net of U1.4 (PC15)
- no-connect marks 0 -> 1
Changed lines of the file:
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@@
 		(color 0 0 0 0)
+	)
+	(no_connect
+		(at 129.54 120.65)
 	)
 	(wire
@@
 			)
 			(justify left)
-		)
-	)
-	(hierarchical_label "LED2"
-		(shape output)
-		(at 129.54 120.65 180)
-		(effects
-			(font
-				(size 1.27 1.27)
-			)
-			(justify right)
 		)
 	)
@@
 		(dnp no)
 		(fields_autoplaced yes)
-		(property "Reference" "C6"
+		(property "Reference" "C4"
 			(at 198.12 35.5599 0)
 			(effects
@@
 			(project "resc"
 				(path "/83aea3b7-5b9b-498e-8d41-e84fae2f87fa/b16235e1-cba7-448a-b9f5-6f75b6848b7e"
-					(reference "C6")
+					(reference "C4")
 					(unit 1)
 				)
@@
 		(dnp no)
 		(fields_autoplaced yes)
-		(property "Reference" "#PWR032"
+		(property "Reference" "#PWR027"
 			(at 125.73 69.85 0)
 			(effects
@@
 			(project "resc"
 				(path "/83aea3b7-5b9b-498e-8d41-e84fae2f87fa/b16235e1-cba7-448a-b9f5-6f75b6848b7e"
-					(reference "#PWR032")
+					(reference "#PWR027")
 					(unit 1)
 				)
@@
 		(dnp no)
 		(fields_autoplaced yes)
-		(property "Reference" "#PWR035"
+		(property "Reference" "#PWR030"
 			(at 151.13 156.21 0)
 			(effects
@@
 			(project "resc"
 				(path "/83aea3b7-5b9b-498e-8d41-e84fae2f87fa/b16235e1-cba7-448a-b9f5-6f75b6848b7e"
-					(reference "#PWR035")
+					(reference "#PWR030")
 					(unit 1)
 				)
@@
 		(dnp no)
 		(fields_autoplaced yes)
-		(property "Reference" "#PWR031"
+		(property "Reference" "#PWR026"
 			(at 114.3 63.5 0)
 			(effects
@@
 			(project "resc"
 				(path "/83aea3b7-5b9b-498e-8d41-e84fae2f87fa/b16235e1-cba7-448a-b9f5-6f75b6848b7e"
-					(reference "#PWR031")
+					(reference "#PWR026")
 					(unit 1)
 				)
@@
 		(dnp no)
 		(fields_autoplaced yes)
-		(property "Reference" "#PWR029"
+		(property "Reference" "#PWR024"
 			(at 187.96 46.99 0)
 			(effects
@@
 			(project "resc"
 				(path "/83aea3b7-5b9b-498e-8d41-e84fae2f87fa/b16235e1-cba7-448a-b9f5-6f75b6848b7e"
-					(reference "#PWR029")
+					(reference "#PWR024")
 					(unit 1)
 				)
@@
 		(dnp no)
 		(fields_autoplaced yes)
-		(property "Reference" "C8"
+		(property "Reference" "C6"
 			(at 223.52 35.5599 0)
 			(effects
@@
 			(project "resc"
 				(path "/83aea3b7-5b9b-498e-8d41-e84fae2f87fa/b16235e1-cba7-448a-b9f5-6f75b6848b7e"
-					(reference "C8")
+					(reference "C6")
 					(unit 1)
 				)
@@
 		(dnp no)
 		(fields_autoplaced yes)
-		(property "Reference" "C5"
+		(property "Reference" "C3"
 			(at 185.42 35.5599 0)
 			(effects
@@
 			(project "resc"
 				(path "/83aea3b7-5b9b-498e-8d41-e84fae2f87fa/b16235e1-cba7-448a-b9f5-6f75b6848b7e"
-					(reference "C5")
+					(reference "C3")
 					(unit 1)
 				)
@@
 		(dnp no)
 		(fields_autoplaced yes)
-		(property "Reference" "C12"
+		(property "Reference" "C10"
 			(at 78.74 74.9299 0)
 			(effects
@@
 			(project "resc"
 				(path "/83aea3b7-5b9b-498e-8d41-e84fae2f87fa/b16235e1-cba7-448a-b9f5-6f75b6848b7e"
-					(reference "C12")
+					(reference "C10")
 					(unit 1)
 				)
@@
 		(dnp no)
 		(fields_autoplaced yes)
-		(property "Reference" "#PWR030"
+		(property "Reference" "#PWR025"
 			(at 151.13 54.61 0)
 			(effects
@@
 			(project "resc"
 				(path "/83aea3b7-5b9b-498e-8d41-e84fae2f87fa/b16235e1-cba7-448a-b9f5-6f75b6848b7e"
-					(reference "#PWR030")
+					(reference "#PWR025")
 					(unit 1)
 				)
@@
 		(dnp no)
 		(fields_autoplaced yes)
-		(property "Reference" "#PWR034"
+		(property "Reference" "#PWR029"
 			(at 114.3 144.78 0)
 			(effects
@@
 			(project "resc"
 				(path "/83aea3b7-5b9b-498e-8d41-e84fae2f87fa/b16235e1-cba7-448a-b9f5-6f75b6848b7e"
-					(reference "#PWR034")
+					(reference "#PWR029")
 					(unit 1)
 				)
@@
 		(dnp no)
 		(fields_autoplaced yes)
-		(property "Reference" "C13"
+		(property "Reference" "C11"
 			(at 99.06 74.9299 0)
 			(effects
@@
 			(project "resc"
 				(path "/83aea3b7-5b9b-498e-8d41-e84fae2f87fa/b16235e1-cba7-448a-b9f5-6f75b6848b7e"
-					(reference "C13")
+					(reference "C11")
 					(unit 1)
 				)
@@
 		(dnp no)
 		(fields_autoplaced yes)
-		(property "Reference" "C7"
+		(property "Reference" "C5"
 			(at 210.82 35.5599 0)
 			(effects
@@
 			(project "resc"
 				(path "/83aea3b7-5b9b-498e-8d41-e84fae2f87fa/b16235e1-cba7-448a-b9f5-6f75b6848b7e"
-					(reference "C7")
+					(reference "C5")
 					(unit 1)
 				)
@@
 		(dnp no)
 		(fields_autoplaced yes)
-		(property "Reference" "C14"
+		(property "Reference" "C12"
 			(at 111.76 133.3499 0)
 			(effects
@@
 			(project "resc"
 				(path "/83aea3b7-5b9b-498e-8d41-e84fae2f87fa/b16235e1-cba7-448a-b9f5-6f75b6848b7e"
-					(reference "C14")
+					(reference "C12")
 					(unit 1)
 				)
@@
 		(dnp no)
 		(fields_autoplaced yes)
-		(property "Reference" "C9"
+		(property "Reference" "C7"
 			(at 236.22 35.5599 0)
 			(effects
@@
 			(project "resc"
 				(path "/83aea3b7-5b9b-498e-8d41-e84fae2f87fa/b16235e1-cba7-448a-b9f5-6f75b6848b7e"
-					(reference "C9")
+					(reference "C7")
 					(unit 1)
 				)
@@
 		(dnp no)
 		(fields_autoplaced yes)
-		(property "Reference" "C15"
+		(property "Reference" "C13"
 			(at 124.46 133.3499 0)
 			(effects
@@
 			(project "resc"
 				(path "/83aea3b7-5b9b-498e-8d41-e84fae2f87fa/b16235e1-cba7-448a-b9f5-6f75b6848b7e"
-					(reference "C15")
+					(reference "C13")
 					(unit 1)
 				)
@@
 		(dnp no)
 		(fields_autoplaced yes)
-		(property "Reference" "#PWR033"
+		(property "Reference" "#PWR028"
 			(at 86.36 90.17 0)
 			(effects
@@
 			(project "resc"
 				(path "/83aea3b7-5b9b-498e-8d41-e84fae2f87fa/b16235e1-cba7-448a-b9f5-6f75b6848b7e"
-					(reference "#PWR033")
+					(reference "#PWR028")
 					(unit 1)
 				)
@@
 		(dnp no)
 		(fields_autoplaced yes)
-		(property "Reference" "C10"
+		(property "Reference" "C8"
 			(at 248.92 35.5599 0)
 			(effects
@@
 			(project "resc"
 				(path "/83aea3b7-5b9b-498e-8d41-e84fae2f87fa/b16235e1-cba7-448a-b9f5-6f75b6848b7e"
-					(reference "C10")
+					(reference "C8")
 					(unit 1)
 				)
@@
 		(dnp no)
 		(fields_autoplaced yes)
-		(property "Reference" "C11"
+		(property "Reference" "C9"
 			(at 118.11 52.0699 0)
 			(effects
@@
 			(project "resc"
 				(path "/83aea3b7-5b9b-498e-8d41-e84fae2f87fa/b16235e1-cba7-448a-b9f5-6f75b6848b7e"
-					(reference "C11")
+					(reference "C9")
 					(unit 1)
 				)
@@
 		(dnp no)
 		(fields_autoplaced yes)
-		(property "Reference" "#PWR028"
+		(property "Reference" "#PWR023"
 			(at 187.96 36.83 0)
 			(effects
@@
 			(project "resc"
 				(path "/83aea3b7-5b9b-498e-8d41-e84fae2f87fa/b16235e1-cba7-448a-b9f5-6f75b6848b7e"
-					(reference "#PWR028")
+					(reference "#PWR023")
 					(unit 1)
 				)
