File: kicad/mcu.kicad_sch (KiCad schematic)
At the start: 13 parts, among them U1 STM32F405RGTx, Y1 8MHz

Commit message: rev3 ordered
Parts:
- renumbered C8 to C10, C9 to C11, C10 to C12, C11 to C13, C12 to C14, C13 to C15, C3 to C5, C4 to C6, C5 to C7, C6 to C8, C7 to C9
Connections:
- net H1: now also U1.37 (PC6); no longer U1.41 (PA8)
- net H2: now also U1.38 (PC7); no longer U1.42 (PA9)
- net H3: now also U1.39 (PC8); no longer U1.43 (PA10)
- net HALL_1: now also U1.41 (PA8); no longer U1.37 (PC6)
- net HALL_2: now also U1.42 (PA9); no longer U1.38 (PC7)
- net HALL_3: now also U1.43 (PA10); no longer U1.39 (PC8)
- net CONN_SW: now reaches U1.4 (PC15)
- net ADC_15 renamed POWER
- net EN_GATE renamed EN_DRV
- no-connect marks 1 -> 0
Changed lines of the file:
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@@
 		(color 0 0 0 0)
-	)
-	(no_connect
-		(at 129.54 120.65)
 	)
 	(wire
@@
 		)
 	)
+	(hierarchical_label "CONN_SW"
+		(shape input)
+		(at 129.54 120.65 180)
+		(effects
+			(font
+				(size 1.27 1.27)
+			)
+			(justify right)
+		)
+	)
 	(hierarchical_label "LED_RED"
 		(shape output)
@@
 	(hierarchical_label "HALL_2"
 		(shape input)
-		(at 129.54 100.33 180)
-		(effects
-			(font
-				(size 1.27 1.27)
-			)
-			(justify right)
+		(at 170.18 82.55 0)
+		(effects
+			(font
+				(size 1.27 1.27)
+			)
+			(justify left)
 		)
 	)
@@
 		)
 	)
-	(hierarchical_label "ADC_15"
-		(shape input)
+	(hierarchical_label "POWER"
+		(shape output)
 		(at 129.54 95.25 180)
 		(effects
@@
 		)
 	)
-	(hierarchical_label "EN_GATE"
+	(hierarchical_label "EN_DRV"
 		(shape output)
 		(at 170.18 115.57 0)
@@
 	(hierarchical_label "HALL_1"
 		(shape input)
-		(at 129.54 97.79 180)
-		(effects
-			(font
-				(size 1.27 1.27)
-			)
-			(justify right)
+		(at 170.18 80.01 0)
+		(effects
+			(font
+				(size 1.27 1.27)
+			)
+			(justify left)
 		)
 	)
@@
 	(hierarchical_label "H1"
 		(shape output)
-		(at 170.18 80.01 0)
-		(effects
-			(font
-				(size 1.27 1.27)
-			)
-			(justify left)
+		(at 129.54 97.79 180)
+		(effects
+			(font
+				(size 1.27 1.27)
+			)
+			(justify right)
 		)
 	)
@@
 	(hierarchical_label "HALL_3"
 		(shape input)
-		(at 129.54 102.87 180)
-		(effects
-			(font
-				(size 1.27 1.27)
-			)
-			(justify right)
+		(at 170.18 85.09 0)
+		(effects
+			(font
+				(size 1.27 1.27)
+			)
+			(justify left)
 		)
 	)
@@
 	(hierarchical_label "H3"
 		(shape output)
-		(at 170.18 85.09 0)
-		(effects
-			(font
-				(size 1.27 1.27)
-			)
-			(justify left)
+		(at 129.54 102.87 180)
+		(effects
+			(font
+				(size 1.27 1.27)
+			)
+			(justify right)
 		)
 	)
@@
 	(hierarchical_label "H2"
 		(shape output)
-		(at 170.18 82.55 0)
-		(effects
-			(font
-				(size 1.27 1.27)
-			)
-			(justify left)
+		(at 129.54 100.33 180)
+		(effects
+			(font
+				(size 1.27 1.27)
+			)
+			(justify right)
 		)
 	)
@@
 		(dnp no)
 		(fields_autoplaced yes)
-		(property "Reference" "C4"
+		(property "Reference" "C6"
 			(at 198.12 35.5599 0)
 			(effects
@@
 			(project "resc"
 				(path "/83aea3b7-5b9b-498e-8d41-e84fae2f87fa/b16235e1-cba7-448a-b9f5-6f75b6848b7e"
-					(reference "C4")
+					(reference "C6")
 					(unit 1)
 				)
@@
 		(dnp no)
 		(fields_autoplaced yes)
-		(property "Reference" "#PWR027"
+		(property "Reference" "#PWR032"
 			(at 125.73 69.85 0)
 			(effects
@@
 			(project "resc"
 				(path "/83aea3b7-5b9b-498e-8d41-e84fae2f87fa/b16235e1-cba7-448a-b9f5-6f75b6848b7e"
-					(reference "#PWR027")
+					(reference "#PWR032")
 					(unit 1)
 				)
@@
 		(dnp no)
 		(fields_autoplaced yes)
-		(property "Reference" "#PWR030"
+		(property "Reference" "#PWR035"
 			(at 151.13 156.21 0)
 			(effects
@@
 			(project "resc"
 				(path "/83aea3b7-5b9b-498e-8d41-e84fae2f87fa/b16235e1-cba7-448a-b9f5-6f75b6848b7e"
-					(reference "#PWR030")
+					(reference "#PWR035")
 					(unit 1)
 				)
@@
 		(dnp no)
 		(fields_autoplaced yes)
-		(property "Reference" "#PWR026"
+		(property "Reference" "#PWR031"
 			(at 114.3 63.5 0)
 			(effects
@@
 			(project "resc"
 				(path "/83aea3b7-5b9b-498e-8d41-e84fae2f87fa/b16235e1-cba7-448a-b9f5-6f75b6848b7e"
-					(reference "#PWR026")
+					(reference "#PWR031")
 					(unit 1)
 				)
@@
 		(dnp no)
 		(fields_autoplaced yes)
-		(property "Reference" "#PWR024"
+		(property "Reference" "#PWR029"
 			(at 187.96 46.99 0)
 			(effects
@@
 			(project "resc"
 				(path "/83aea3b7-5b9b-498e-8d41-e84fae2f87fa/b16235e1-cba7-448a-b9f5-6f75b6848b7e"
-					(reference "#PWR024")
+					(reference "#PWR029")
 					(unit 1)
 				)
@@
 		(dnp no)
 		(fields_autoplaced yes)
-		(property "Reference" "C6"
+		(property "Reference" "C8"
 			(at 223.52 35.5599 0)
 			(effects
@@
 			(project "resc"
 				(path "/83aea3b7-5b9b-498e-8d41-e84fae2f87fa/b16235e1-cba7-448a-b9f5-6f75b6848b7e"
-					(reference "C6")
+					(reference "C8")
 					(unit 1)
 				)
@@
 		(dnp no)
 		(fields_autoplaced yes)
-		(property "Reference" "C3"
+		(property "Reference" "C5"
 			(at 185.42 35.5599 0)
 			(effects
@@
 			(project "resc"
 				(path "/83aea3b7-5b9b-498e-8d41-e84fae2f87fa/b16235e1-cba7-448a-b9f5-6f75b6848b7e"
-					(reference "C3")
+					(reference "C5")
 					(unit 1)
 				)
@@
 		(dnp no)
 		(fields_autoplaced yes)
-		(property "Reference" "C10"
+		(property "Reference" "C12"
 			(at 78.74 74.9299 0)
 			(effects
@@
 			(project "resc"
 				(path "/83aea3b7-5b9b-498e-8d41-e84fae2f87fa/b16235e1-cba7-448a-b9f5-6f75b6848b7e"
-					(reference "C10")
+					(reference "C12")
 					(unit 1)
 				)
@@
 		(dnp no)
 		(fields_autoplaced yes)
-		(property "Reference" "#PWR025"
+		(property "Reference" "#PWR030"
 			(at 151.13 54.61 0)
 			(effects
@@
 			(project "resc"
 				(path "/83aea3b7-5b9b-498e-8d41-e84fae2f87fa/b16235e1-cba7-448a-b9f5-6f75b6848b7e"
-					(reference "#PWR025")
+					(reference "#PWR030")
 					(unit 1)
 				)
@@
 		(dnp no)
 		(fields_autoplaced yes)
-		(property "Reference" "#PWR029"
+		(property "Reference" "#PWR034"
 			(at 114.3 144.78 0)
 			(effects
@@
 			(project "resc"
 				(path "/83aea3b7-5b9b-498e-8d41-e84fae2f87fa/b16235e1-cba7-448a-b9f5-6f75b6848b7e"
-					(reference "#PWR029")
+					(reference "#PWR034")
 					(unit 1)
 				)
@@
 		(dnp no)
 		(fields_autoplaced yes)
-		(property "Reference" "C11"
+		(property "Reference" "C13"
 			(at 99.06 74.9299 0)
 			(effects
@@
 			(project "resc"
 				(path "/83aea3b7-5b9b-498e-8d41-e84fae2f87fa/b16235e1-cba7-448a-b9f5-6f75b6848b7e"
-					(reference "C11")
+					(reference "C13")
 					(unit 1)
 				)
@@
 		(dnp no)
 		(fields_autoplaced yes)
-		(property "Reference" "C5"
+		(property "Reference" "C7"
 			(at 210.82 35.5599 0)
 			(effects
@@
 			(project "resc"
 				(path "/83aea3b7-5b9b-498e-8d41-e84fae2f87fa/b16235e1-cba7-448a-b9f5-6f75b6848b7e"
-					(reference "C5")
+					(reference "C7")
 					(unit 1)
 				)
@@
 		(dnp no)
 		(fields_autoplaced yes)
-		(property "Reference" "C12"
+		(property "Reference" "C14"
 			(at 111.76 133.3499 0)
 			(effects
@@
 			(project "resc"
 				(path "/83aea3b7-5b9b-498e-8d41-e84fae2f87fa/b16235e1-cba7-448a-b9f5-6f75b6848b7e"
-					(reference "C12")
+					(reference "C14")
 					(unit 1)
 				)
@@
 		(dnp no)
 		(fields_autoplaced yes)
-		(property "Reference" "C7"
+		(property "Reference" "C9"
 			(at 236.22 35.5599 0)
 			(effects
@@
 			(project "resc"
 				(path "/83aea3b7-5b9b-498e-8d41-e84fae2f87fa/b16235e1-cba7-448a-b9f5-6f75b6848b7e"
-					(reference "C7")
+					(reference "C9")
 					(unit 1)
 				)
@@
 		(dnp no)
 		(fields_autoplaced yes)
-		(property "Reference" "C13"
+		(property "Reference" "C15"
 			(at 124.46 133.3499 0)
 			(effects
@@
 			(project "resc"
 				(path "/83aea3b7-5b9b-498e-8d41-e84fae2f87fa/b16235e1-cba7-448a-b9f5-6f75b6848b7e"
-					(reference "C13")
+					(reference "C15")
 					(unit 1)
 				)
@@
 		(dnp no)
 		(fields_autoplaced yes)
-		(property "Reference" "#PWR028"
+		(property "Reference" "#PWR033"
 			(at 86.36 90.17 0)
 			(effects
@@
 			(project "resc"
 				(path "/83aea3b7-5b9b-498e-8d41-e84fae2f87fa/b16235e1-cba7-448a-b9f5-6f75b6848b7e"
-					(reference "#PWR028")
+					(reference "#PWR033")
 					(unit 1)
 				)
@@
 		(dnp no)
 		(fields_autoplaced yes)
-		(property "Reference" "C8"
+		(property "Reference" "C10"
 			(at 248.92 35.5599 0)
 			(effects
@@
 			(project "resc"
 				(path "/83aea3b7-5b9b-498e-8d41-e84fae2f87fa/b16235e1-cba7-448a-b9f5-6f75b6848b7e"
-					(reference "C8")
+					(reference "C10")
 					(unit 1)
 				)
@@
 		(dnp no)
 		(fields_autoplaced yes)
-		(property "Reference" "C9"
+		(property "Reference" "C11"
 			(at 118.11 52.0699 0)
 			(effects
@@
 			(project "resc"
 				(path "/83aea3b7-5b9b-498e-8d41-e84fae2f87fa/b16235e1-cba7-448a-b9f5-6f75b6848b7e"
-					(reference "C9")
+					(reference "C11")
 					(unit 1)
 				)
@@
 		(dnp no)
 		(fields_autoplaced yes)
-		(property "Reference" "#PWR023"
+		(property "Reference" "#PWR028"
 			(at 187.96 36.83 0)
 			(effects
@@
 			(project "resc"
 				(path "/83aea3b7-5b9b-498e-8d41-e84fae2f87fa/b16235e1-cba7-448a-b9f5-6f75b6848b7e"
-					(reference "#PWR023")
+					(reference "#PWR028")
 					(unit 1)
 				)
